File: guitar_tuner/untitled.kicad_sch2.kicad_sch (KiCad schematic)
At the start: 0 parts

Commit message: Buzzer Circuit
Transistor and buzzer, have not yet set up power or connected to ESP32
Parts:
- added BZ1: Buzzer, symbol Device:Buzzer
- added Q1: NPN, symbol Simulation_SPICE:NPN
- added R5: 1k, symbol Device:R
Connections:
- new net: BZ1.2 (-), Q1.1 (C)
- new net: Q1.2 (B), R5.2
- new net GND: Q1.3 (E)
