File: guitar_tuner/untitled.kicad_sch1.kicad_sch (KiCad schematic)
At the start: 0 parts

Commit message: LED
Addition of LED Circuits
Parts:
- added D1, D2, D3: LED, symbol Device:LED
- added R2, R3, R4: 330, symbol Device:R
Connections:
- new net: D2.2 (A), R3.2
- new net: D1.2 (A), R2.2
- new net: D3.2 (A), R4.2
- new net GND: D1.1 (K), D2.1 (K), D3.1 (K)
- new net LED_GREEN: R4.1
- new net LED_RED: R2.1
- new net LED_YELLOW: R3.1

Commit message: Led Circuit Footprints
Parts:
- D1, D2, D3: footprint (none) -> LED_SMD:LED_0805_2012Metric_Pad1.15x1.40mm_HandSolder
- R2, R3, R4: footprint (none) -> Resistor_SMD:R_0805_2012Metric_Pad1.20x1.40mm_HandSolder
Changed lines of the file:
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@@
 			)
 		)
-		(property "Footprint" ""
+		(property "Footprint" "Resistor_SMD:R_0805_2012Metric_Pad1.20x1.40mm_HandSolder"
 			(at 88.392 81.28 90)
 			(effects
@@
 			)
 		)
-		(property "Footprint" ""
+		(property "Footprint" "Resistor_SMD:R_0805_2012Metric_Pad1.20x1.40mm_HandSolder"
 			(at 68.072 81.28 90)
 			(effects
@@
 			)
 		)
-		(property "Footprint" ""
+		(property "Footprint" "LED_SMD:LED_0805_2012Metric_Pad1.15x1.40mm_HandSolder"
 			(at 110.49 93.98 0)
 			(effects
@@
 			)
 		)
-		(property "Footprint" ""
+		(property "Footprint" "Resistor_SMD:R_0805_2012Metric_Pad1.20x1.40mm_HandSolder"
 			(at 108.712 81.28 90)
 			(effects
@@
 			)
 		)
-		(property "Footprint" ""
+		(property "Footprint" "LED_SMD:LED_0805_2012Metric_Pad1.15x1.40mm_HandSolder"
 			(at 90.17 93.98 0)
 			(effects
@@
 			)
 		)
-		(property "Footprint" ""
+		(property "Footprint" "LED_SMD:LED_0805_2012Metric_Pad1.15x1.40mm_HandSolder"
 			(at 69.85 93.98 0)
 			(effects
